Commit message: final

File: robot_arm_description/urdf/robot_arm.urdf.xacro (robot description, xacro)
@@ -180,8 +180,7 @@
         <mesh filename="package://robot_arm_description/meshes/gripper_base.stl" scale="0.001 0.001 0.001"/>
       </geometry>
-      <material
-        name="">
-        <color rgba="0.79216 0.81961 0.93333 1" />
-      </material>
+      <material name="gripper_grey">
+        <color rgba="0.5 0.5 0.5 1.0"/>
+    </material>
     </visual>
     <collision>
@@ -219,4 +218,7 @@
           <mesh filename="package://robot_arm_description/meshes/right_gear.stl" scale="0.001 0.001 0.001" />
       </geometry>
+      <material name="gripper_grey">
+          <color rgba="0.5 0.5 0.5 1.0"/>
+      </material>
     </visual>
     <collision name="right_gear_collision">
@@ -254,4 +256,7 @@
             <mesh filename="package://robot_arm_description/meshes/links.stl" scale="0.001 0.001 0.001" />
         </geometry>
+        <material name="gripper_grey">
+            <color rgba="0.5 0.5 0.5 1.0"/>
+        </material>
     </visual>
     <collision name="links_collision">
@@ -290,4 +295,7 @@
           <mesh filename="package://robot_arm_description/meshes/gripper-fingures.stl" scale="0.001 0.001 0.001" />
       </geometry>
+      <material name="gripper_grey">
+        <color rgba="0.5 0.5 0.5 1.0"/>
+    </material>
     </visual>
     <collision>
@@ -326,4 +334,7 @@
           <mesh filename="package://robot_arm_description/meshes/left_gear.stl" scale="0.001 0.001 0.001" />
       </geometry>
+      <material name="gripper_grey">
+        <color rgba="0.5 0.5 0.5 1.0"/>
+    </material>
   </visual>
     <collision>
@@ -362,5 +373,11 @@
           <mesh filename="package://robot_arm_description/meshes/links.stl" scale="0.001 0.001 0.001" />
       </geometry>
-    </visual>
+      <material name="gripper_grey">
+        <color rgba="0.5 0.5 0.5 1.0"/>
+      </material>
+    </visual>
+    <material name="gripper_grey">
+        <color rgba="0.5 0.5 0.5 1.0"/>
+    </material>
     <collision>
       <origin xyz="0.0 0.0 -0.0087" rpy="0.0 0.0 0.031416" />
@@ -398,4 +415,7 @@
           <mesh filename="package://robot_arm_description/meshes/gripper-fingures.stl" scale="0.001 0.001 0.001" />
       </geometry>
+      <material name="gripper_grey">
+        <color rgba="0.5 0.5 0.5 1.0"/>
+    </material>
     </visual>
     <collision name="gripper-fingures_collision">
